File: hardware/radio.kicad_sch (KiCad schematic)
At the start: 22 parts

Commit message: schematic
Parts:
- removed J?: USB_C_Receptacle_USB2.0, symbol Connector:USB_C_Receptacle_USB2.0
- added C5: 56n, Capacitor_SMD:C_0603_1608Metric, symbol Device:C
- added C6: 5n6, Capacitor_SMD:C_0603_1608Metric, symbol Device:C
- added J1: 105450-0101, wyswietlacze:MOLEX_105450-0101, symbol 105450-0101:105450-0101
- added R4: 5k6, Resistor_SMD:R_0603_1608Metric, symbol Device:R
- C1, C10, C11, C12, C2, C3: renamed from C?; footprint (none) -> Capacitor_SMD:C_1206_3216Metric
- C4, C7, C8: renamed from C?; footprint (none) -> Capacitor_SMD:C_0603_1608Metric
- C9: renamed from C?; value 0.1u -> 100n; footprint (none) -> Capacitor_SMD:C_0603_1608Metric
- J2, J3: renamed from J?; footprint (none) -> Connector_PinHeader_2.54mm:PinHeader_1x02_P2.54mm_Vertical
- L1: renamed from L?; footprint (none) -> wyswietlacze:L_2010Metric; Sklep (none) -> https://www.mouser.pl/ProductDetail/Bourns/SRP2010TMA-2R2M?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
- R1, R2: footprint (none) -> Resistor_SMD:R_0603_1608Metric
- R3: renamed from R?; footprint (none) -> Resistor_SMD:R_0603_1608Metric
- gave numbers to parts that had none: 5
Connections:
- net -BATT: now also C5.2, C6.2
- net at U3.6 (COMP): now also C5.1, R4.1
- new net: C6.1, R4.2
- new net: J1.A1 (GND_A), J1.A12 (GND_A)
- new net: J1.A4 (VBUS_A), J1.A9 (VBUS_A)
- new net: J1.B1 (GND_B), J1.B12 (GND_B)
- new net: J1.B4 (VBUS_B), J1.B9 (VBUS_B)
- new net: J1.S1 (SHIELD), J1.S2 (SHIELD), J1.S3 (SHIELD), J1.S4 (SHIELD)
Other:
- moved on the sheet: C10, C3, C4, C9, J3, U2, U4
