File: hardware/radio.kicad_sch (KiCad schematic)
At the start: 60 parts, among them J1 105450-0101, J2 Conn_01x02, J3 Conn_01x02, J4 Conn_01x04, J5 Conn_01x02_Male, Q1 Q_PMOS_DGS, Q2 Q_NMOS_DGS, Q3 Q_NMOS_DGS, Q4 Q_PMOS_DGS, SW1 SW_BOOT, SW2 SW_RST, SW3 SW_1, SW4 Rot_Enc, SW5 SW_2, SW6 SW_3, SW7 SW_PWR, U1 TP4056, U2 ESP32-WROOM-32, U3 TPS5432, U4 MAX98357

Commit message: began placement
Parts:
- added R21: 0, Resistor_SMD:R_0603_1608Metric, symbol Device:R
- Q3: Sklep (none) -> https://kamami.pl/z-kanalem-typu-n/231862-ao3402.html
- Q4: Sklep (none) -> https://kamami.pl/z-kanalem-typu-p/231026-ao3401.html
- SW1, SW2, SW3, SW5, SW6, SW7: footprint (none) -> Button_Switch_SMD:SW_Push_1P1T_NO_6x6mm_H9.5mm
Connections:
- net ENC_BTN: now also R21.2
- net at D1.1 (K), D2.1 (K), SW7.2: now also R21.1
- net -BATT renamed GND
Changed lines of the file:
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@@
   (junction (at 149.86 22.86) (diameter 0) (color 0 0 0 0)
   )
-  (junction (at 69.85 25.4) (diameter 0) (color 0 0 0 0)
-  )
   (junction (at 243.84 39.37) (diameter 0) (color 0 0 0 0)
   )
@@
     (stroke (width 0) (type default) (color 0 0 0 0))
   )
-  (wire (pts (xy 69.85 20.32) (xy 69.85 25.4))
-    (stroke (width 0) (type default) (color 0 0 0 0))
-  )
   (wire (pts (xy 214.63 39.37) (xy 215.9 39.37))
     (stroke (width 0) (type default) (color 0 0 0 0))
@@
     (stroke (width 0) (type default) (color 0 0 0 0))
   )
-  (wire (pts (xy 69.85 25.4) (xy 71.12 25.4))
+  (wire (pts (xy 68.58 25.4) (xy 71.12 25.4))
     (stroke (width 0) (type default) (color 0 0 0 0))
   )
@@
   )
   (wire (pts (xy 100.33 166.37) (xy 100.33 167.64))
-    (stroke (width 0) (type default) (color 0 0 0 0))
-  )
-  (wire (pts (xy 68.58 25.4) (xy 69.85 25.4))
     (stroke (width 0) (type default) (color 0 0 0 0))
   )
@@
     )
   )
+  (global_label "ENC_BTN" (shape input) (at 147.32 44.45 0) (fields_autoplaced)
+    (effects (font (size 1.27 1.27)) (justify left))
+    (property "Intersheet References" "${INTERSHEET_REFS}" (id 0) (at 158.0183 44.3706 0)
+      (effects (font (size 1.27 1.27)) (justify left) hide)
+    )
+  )
   (global_label "BTN_2" (shape input) (at 113.03 166.37 180) (fields_autoplaced)
     (effects (font (size 1.27 1.27)) (justify right))
@@
       (effects (font (size 1.27 1.27)) (justify left))
     )
-    (property "Footprint" "" (id 2) (at 105.41 172.72 0)
+    (property "Footprint" "Button_Switch_SMD:SW_Push_1P1T_NO_6x6mm_H9.5mm" (id 2) (at 105.41 172.72 0)
       (effects (font (size 1.27 1.27)) hide)
     )
@@
       (effects (font (size 1.27 1.27)) (justify right))
     )
-    (property "Footprint" "" (id 2) (at 116.84 97.79 0)
+    (property "Footprint" "Button_Switch_SMD:SW_Push_1P1T_NO_6x6mm_H9.5mm" (id 2) (at 116.84 97.79 0)
       (effects (font (size 1.27 1.27)) hide)
     )
@@
     (property "Reference" "SW1" (id 0) (at 173.99 82.55 0))
     (property "Value" "SW_BOOT" (id 1) (at 173.99 85.09 0))
-    (property "Footprint" "" (id 2) (at 173.99 85.09 0)
+    (property "Footprint" "Button_Switch_SMD:SW_Push_1P1T_NO_6x6mm_H9.5mm" (id 2) (at 173.99 85.09 0)
       (effects (font (size 1.27 1.27)) hide)
     )
@@
     (pin "1")
     (pin "2")
-  )
-  (symbol (lib_id "power:-BATT") (at 69.85 20.32 0) (unit 1)
-    (in_bom yes) (on_board yes) (fields_autoplaced)
-    (property "Reference" "#PWR0115" (id 0) (at 69.85 24.13 0)
-      (effects (font (size 1.27 1.27)) hide)
-    )
-    (property "Value" "-BATT" (id 1) (at 69.85 15.24 0))
-    (property "Footprint" "" (id 2) (at 69.85 20.32 0)
-      (effects (font (size 1.27 1.27)) hide)
-    )
-    (property "Datasheet" "" (id 3) (at 69.85 20.32 0)
-      (effects (font (size 1.27 1.27)) hide)
-    )
-    (pin "1")
   )
   (symbol (lib_id "Device:C") (at 179.07 50.8 0) (unit 1)
@@
       (effects (font (size 1.27 1.27)) (justify left))
     )
-    (property "Footprint" "" (id 2) (at 120.65 172.72 0)
+    (property "Footprint" "Button_Switch_SMD:SW_Push_1P1T_NO_6x6mm_H9.5mm" (id 2) (at 120.65 172.72 0)
       (effects (font (size 1.27 1.27)) hide)
     )
@@
     (pin "1")
   )
+  (symbol (lib_id "Device:R") (at 143.51 44.45 90) (unit 1)
+    (in_bom yes) (on_board yes) (fields_autoplaced)
+    (property "Reference" "R21" (id 0) (at 143.51 38.1 90))
+    (property "Value" "0" (id 1) (at 143.51 40.64 90))
+    (property "Footprint" "Resistor_SMD:R_0603_1608Metric" (id 2) (at 143.51 46.228 90)
+      (effects (font (size 1.27 1.27)) hide)
+    )
+    (property "Datasheet" "~" (id 3) (at 143.51 44.45 0)
+      (effects (font (size 1.27 1.27)) hide)
+    )
+    (pin "1")
+    (pin "2")
+  )
   (symbol (lib_id "power:+3V3") (at 90.17 105.41 0) (unit 1)
     (in_bom yes) (on_board yes) (fields_autoplaced)
@@
       (effects (font (size 1.27 1.27)) (justify left))
     )
-    (property "Footprint" "" (id 2) (at 134.62 172.72 0)
+    (property "Footprint" "Button_Switch_SMD:SW_Push_1P1T_NO_6x6mm_H9.5mm" (id 2) (at 134.62 172.72 0)
       (effects (font (size 1.27 1.27)) hide)
     )
@@
       (effects (font (size 1.27 1.27)) hide)
     )
+    (property "Sklep" "https://kamami.pl/z-kanalem-typu-p/231026-ao3401.html" (id 4) (at 124.46 34.29 90)
+      (effects (font (size 1.27 1.27)) hide)
+    )
     (pin "1")
     (pin "2")
@@
     )
     (property "Datasheet" "~" (id 3) (at 121.92 50.8 0)
+      (effects (font (size 1.27 1.27)) hide)
+    )
+    (property "Sklep" "https://kamami.pl/z-kanalem-typu-n/231862-ao3402.html" (id 4) (at 121.92 50.8 0)
       (effects (font (size 1.27 1.27)) hide)
     )
@@
       (effects (font (size 1.27 1.27)) (justify left))
     )
-    (property "Footprint" "" (id 2) (at 144.78 52.07 0)
+    (property "Footprint" "Button_Switch_SMD:SW_Push_1P1T_NO_6x6mm_H9.5mm" (id 2) (at 144.78 52.07 0)
       (effects (font (size 1.27 1.27)) hide)
     )
@@
       (reference "#PWR0114") (unit 1) (value "+3V3") (footprint "")
     )
-    (path "/3fc451b2-19ba-4fee-a577-06d70b0c7e03"
-      (reference "#PWR0115") (unit 1) (value "-BATT") (footprint "")
-    )
     (path "/ec09260e-946a-4d95-8812-f92989b6ac9f"
       (reference "#PWR0116") (unit 1) (value "+5V") (footprint "")
@@
       (reference "R20") (unit 1) (value "10k") (footprint "Resistor_SMD:R_0603_1608Metric")
     )
+    (path "/72963581-de2e-4b07-8d6a-1a74adeb50f0"
+      (reference "R21") (unit 1) (value "0") (footprint "Resistor_SMD:R_0603_1608Metric")
+    )
     (path "/395dc202-ab89-4816-9a78-379ff056d9ef"
-      (reference "SW1") (unit 1) (value "SW_BOOT") (footprint "")
+      (reference "SW1") (unit 1) (value "SW_BOOT") (footprint "Button_Switch_SMD:SW_Push_1P1T_NO_6x6mm_H9.5mm")
     )
     (path "/12a57ffb-27dd-4e5a-be57-6d9aafe8ec82"
-      (reference "SW2") (unit 1) (value "SW_RST") (footprint "")
+      (reference "SW2") (unit 1) (value "SW_RST") (footprint "Button_Switch_SMD:SW_Push_1P1T_NO_6x6mm_H9.5mm")
     )
     (path "/10988266-4f97-410b-b13a-7a0f429aa8dd"
-      (reference "SW3") (unit 1) (value "SW_1") (footprint "")
+      (reference "SW3") (unit 1) (value "SW_1") (footprint "Button_Switch_SMD:SW_Push_1P1T_NO_6x6mm_H9.5mm")
     )
     (path "/91639b42-c470-42c9-9909-45f7e876089b"
@@
     )
     (path "/6ac18683-c83a-4313-895c-f36b2e45fa74"
-      (reference "SW5") (unit 1) (value "SW_2") (footprint "")
+      (reference "SW5") (unit 1) (value "SW_2") (footprint "Button_Switch_SMD:SW_Push_1P1T_NO_6x6mm_H9.5mm")
     )
     (path "/7583a15e-5ed1-4fdd-88e8-b23249c693fe"
-      (reference "SW6") (unit 1) (value "SW_3") (footprint "")
+      (reference "SW6") (unit 1) (value "SW_3") (footprint "Button_Switch_SMD:SW_Push_1P1T_NO_6x6mm_H9.5mm")
     )
     (path "/e887eda6-a382-43f6-9c8f-b443c1d607f0"
-      (reference "SW7") (unit 1) (value "SW_PWR") (footprint "")
+      (reference "SW7") (unit 1) (value "SW_PWR") (footprint "Button_Switch_SMD:SW_Push_1P1T_NO_6x6mm_H9.5mm")
     )
     (path "/a274958a-ae53-4989-b48b-9f41b3964f32"

Commit message: placement
Parts:
- removed R21: 0, Resistor_SMD:R_0603_1608Metric, symbol Device:R
- removed SW7: SW_PWR, Button_Switch_SMD:SW_Push_1P1T_NO_6x6mm_H9.5mm, symbol Switch:SW_Push
- R16: value 10k -> 0
Connections:
- net PWR_READ is gone; now on net ENC_BTN: D1.2 (A), R20.2
- net +3V3: no longer R16.1
- net ENC_BTN: now also R16.1; no longer R16.2, SW4.S1
- net ENC_S1: now reaches D1.1 (K), D2.1 (K)
- net ENC_S1: now also R16.2, SW4.S1

Commit message: placement (possibly close to final)
Connections:
- no-connect marks 0 -> 6
Changed lines of the file:
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@@
   (junction (at 161.29 22.86) (diameter 0) (color 0 0 0 0)
   )
+  (no_connect (at 132.08 130.81))
+  (no_connect (at 132.08 133.35))
+  (no_connect (at 132.08 120.65))
+  (no_connect (at 132.08 123.19))
+  (no_connect (at 132.08 125.73))
+  (no_connect (at 132.08 128.27))
   (wire (pts (xy 58.42 152.4) (xy 58.42 156.21))
     (stroke (width 0) (type default) (color 0 0 0 0))
@@
     )
     (property "Datasheet" "~" (id 3) (at 76.2 22.86 0)
-      (effects (font (size 1.27 1.27)) hide)
-    )
-    (pin "1")
-    (pin "2")
-  )
-  (symbol (lib_id "Connector:Conn_01x02_Male") (at 125.73 16.51 270) (unit 1)
-    (in_bom yes) (on_board yes) (fields_autoplaced)
-    (property "Reference" "J5" (id 0) (at 127 15.8749 90)
-      (effects (font (size 1.27 1.27)) (justify left))
-    )
-    (property "Value" "Conn_01x02_Male" (id 1) (at 127 18.4149 90)
-      (effects (font (size 1.27 1.27)) (justify left))
-    )
-    (property "Footprint" "Connector_PinHeader_2.54mm:PinHeader_1x02_P2.54mm_Horizontal" (id 2) (at 125.73 16.51 0)
-      (effects (font (size 1.27 1.27)) hide)
-    )
-    (property "Datasheet" "~" (id 3) (at 125.73 16.51 0)
       (effects (font (size 1.27 1.27)) hide)
     )
@@
     )
     (pin "1")
+  )
+  (symbol (lib_id "Connector:Conn_01x02_Male") (at 125.73 16.51 270) (unit 1)
+    (in_bom yes) (on_board yes) (fields_autoplaced)
+    (property "Reference" "J5" (id 0) (at 127 15.8749 90)
+      (effects (font (size 1.27 1.27)) (justify left))
+    )
+    (property "Value" "Conn_01x02_Male" (id 1) (at 127 18.4149 90)
+      (effects (font (size 1.27 1.27)) (justify left))
+    )
+    (property "Footprint" "Connector_PinHeader_2.54mm:PinHeader_1x02_P2.54mm_Horizontal" (id 2) (at 125.73 16.51 0)
+      (effects (font (size 1.27 1.27)) hide)
+    )
+    (property "Datasheet" "~" (id 3) (at 125.73 16.51 0)
+      (effects (font (size 1.27 1.27)) hide)
+    )
+    (pin "1")
+    (pin "2")
   )
   (symbol (lib_id "Device:R") (at 115.57 161.29 0) (unit 1)
@@
       (reference "J4") (unit 1) (value "Conn_01x04") (footprint "Connector_PinHeader_2.54mm:PinHeader_1x04_P2.54mm_Vertical")
     )
-    (path "/09b8ca6d-45e5-4557-b590-29cd6663a0a8"
+    (path "/acee5406-a5db-4211-8402-727fd651d45d"
       (reference "J5") (unit 1) (value "Conn_01x02_Male") (footprint "Connector_PinHeader_2.54mm:PinHeader_1x02_P2.54mm_Horizontal")
     )

Commit message: routing
Parts:
- added R21, R22: 100k, Resistor_SMD:R_0603_1608Metric, symbol Device:R
Connections:
- net +3V3: now also R21.2
- net ADC IN: now also U2.24 (IO2)
- net ADC_ENABLE: now also U2.23 (IO15)
- net ENC_BTN: now also U2.16 (IO13)
- net GND: now also R22.2
- net I2S_DIN: now reaches U4.1 (DIN)
- net I2S_DIN: now also U2.12 (IO27)
- net I2S_LRCLK: now reaches U4.14 (LRCLK)
- net I2S_LRCLK: now also U2.14 (IO12)
- net I2S_BCLK: now reaches U4.16 (BCLK)
- net I2S_BCLK: now also U2.13 (IO14)
- net at U4.2 (GAIN_SLOT): now also R21.1, R22.1
- net I2S_SD_MODE: now reaches U4.4 (SD_MODE)
- net I2S_SD_MODE: now also U2.11 (IO26)
Other:
- moved on the sheet: DISP1
