File: hardware/radio.kicad_pcb (KiCad board)
At the start: 2 copper layers, 7.3 x 9.3 mm, 25 parts, among them J1 105450-0101, J2 Conn_01x02, J3 Conn_01x02, U1 TP4056, U2 ESP32-WROOM-32, U3 TPS5432, U4 MAX98357

Commit message: schematic
Parts:
- added C13: 100n, Capacitor_SMD:C_0603_1608Metric, F.Cu at (118.0, 37.0)
- added C14: 10u, Capacitor_SMD:C_1206_3216Metric, F.Cu at (113.2, 37.4)
- added J4: Conn_01x04, Connector_PinHeader_2.54mm:PinHeader_1x04_P2.54mm_Vertical, F.Cu at (108.0, 38.1)
Connections:
- net GND renamed -BATT
- U2 pad 3: unconnected-(U2-Pad3) -> +3V3
- U2 pad 34: unconnected-(U2-Pad34) -> Net-(U2-Pad34)
- U2 pad 35: unconnected-(U2-Pad35) -> Net-(U2-Pad35)

Commit message: began placement
Parts:
- added C15: 100n, Capacitor_SMD:C_0603_1608Metric, F.Cu at (60.0, 38.0)
- added C16: 100n, Capacitor_SMD:C_0603_1608Metric, F.Cu at (95.0, 46.0)
- added D1: D_Schottky, Diode_SMD:D_SMA, F.Cu at (58.0, 60.0)
- added D2: D_Schottky, Diode_SMD:D_SMA, F.Cu at (56.0, 66.0)
- added J5: Conn_01x02_Male, Connector_PinHeader_2.54mm:PinHeader_1x02_P2.54mm_Horizontal, F.Cu at (35.4, 56.3)
- added Q1: Q_PMOS_DGS, Package_TO_SOT_SMD:SOT-23, F.Cu at (49.1, 48.0)
- added Q2: Q_NMOS_DGS, Package_TO_SOT_SMD:SOT-23, F.Cu at (53.0, 46.0)
- added Q3: Q_NMOS_DGS, Package_TO_SOT_SMD:SOT-23, F.Cu at (54.0, 70.1)
- added Q4: Q_PMOS_DGS, Package_TO_SOT_SMD:SOT-23, F.Cu at (50.0, 72.0)
- added R10: 5k1, Resistor_SMD:R_0603_1608Metric, F.Cu at (39.2, 38.0)
- added R11: 10k, Resistor_SMD:R_0603_1608Metric, F.Cu at (110.9, 67.0)
- added R12: 10k, Resistor_SMD:R_0603_1608Metric, F.Cu at (114.0, 103.0)
- added R13: 10k, Resistor_SMD:R_0603_1608Metric, F.Cu at (104.9, 67.0)
- added R14: 10k, Resistor_SMD:R_0603_1608Metric, F.Cu at (112.0, 112.0)
- added R15: 10k, Resistor_SMD:R_0603_1608Metric, F.Cu at (115.0, 124.0)
- added R16: 10k, Resistor_SMD:R_0603_1608Metric, F.Cu at (101.9, 49.0)
- added R17: 10k, Resistor_SMD:R_0603_1608Metric, F.Cu at (58.0, 69.0)
- added R18: 100, Resistor_SMD:R_0603_1608Metric, F.Cu at (58.0, 71.0)
- added R19: 10k, Resistor_SMD:R_0603_1608Metric, F.Cu at (50.0, 69.0)
- added R20: 10k, Resistor_SMD:R_0603_1608Metric, F.Cu at (57.2, 55.2)
- added R21: 0, Resistor_SMD:R_0603_1608Metric, F.Cu at (104.9, 46.0)
- added R5: 10k, Resistor_SMD:R_0603_1608Metric, F.Cu at (60.0, 35.0)
- added R6: 100k, Resistor_SMD:R_0603_1608Metric, F.Cu at (53.0, 49.0)
- added R7: 330k, Resistor_SMD:R_0603_1608Metric, F.Cu at (56.0, 48.0)
- added R8: 10k, Resistor_SMD:R_0603_1608Metric, F.Cu at (49.0, 45.0)
- added R9: 5k1, Resistor_SMD:R_0603_1608Metric, F.Cu at (40.5, 35.7)
- added SW1: SW_BOOT, Button_Switch_SMD:SW_Push_1P1T_NO_6x6mm_H9.5mm, F.Cu at (91.0, 51.0)
- added SW2: SW_RST, Button_Switch_SMD:SW_Push_1P1T_NO_6x6mm_H9.5mm, F.Cu at (54.0, 34.0)
- added SW3: SW_1, Button_Switch_SMD:SW_Push_1P1T_NO_6x6mm_H9.5mm, F.Cu at (108.0, 106.0)
- added SW4: Rot_Enc, Rotary_Encoder:RotaryEncoder_Alps_EC12E-Switch_Vertical_H20mm_CircularMountingHoles, F.Cu at (105.4, 64.2)
- added SW5: SW_2, Button_Switch_SMD:SW_Push_1P1T_NO_6x6mm_H9.5mm, F.Cu at (108.0, 117.0)
- added SW6: SW_3, Button_Switch_SMD:SW_Push_1P1T_NO_6x6mm_H9.5mm, F.Cu at (108.0, 126.0)
- added SW7: SW_PWR, Button_Switch_SMD:SW_Push_1P1T_NO_6x6mm_H9.5mm, F.Cu at (59.0, 118.0)
- moved C8 151.6 mm to (39.2, 60.4), turned to -90 degrees
- moved R2 151.3 mm to (47.0, 56.0)
- moved C12 149.7 mm to (49.0, 59.0), turned to 180 degrees
- moved U3 148.1 mm to (43.2, 58.4)
- moved R1 147.8 mm to (49.0, 56.0)
- moved C11 147.4 mm to (49.0, 61.8), turned to 180 degrees
- moved L1 147.2 mm to (45.0, 64.0), turned to 0 degrees
- moved J1 90.8 mm to (34.0, 36.0), turned to -90 degrees
- moved R3 85.6 mm to (44.0, 34.0)
- moved C5 80.4 mm to (43.9, 52.7), turned to 90 degrees
- moved C1 80.0 mm to (39.9, 32.5), turned to 90 degrees
- moved C7 78.7 mm to (41.2, 52.4), turned to 90 degrees
- moved C4 78.7 mm to (42.2, 63.4), turned to 180 degrees
- moved C2 75.2 mm to (37.9, 46.0), turned to 180 degrees
- moved J2 73.2 mm to (32.0, 48.0), turned to 180 degrees
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Connections:
- C1 pad 2: -BATT -> GND
- C10 pad 1: -BATT -> GND
- C11 pad 2: -BATT -> GND
- C12 pad 2: -BATT -> GND
- C13 pad 1: -BATT -> GND
- C14 pad 1: -BATT -> GND
- C2 pad 2: -BATT -> GND
- C3 pad 1: +BATT -> Net-(C3-Pad1)
- C3 pad 2: -BATT -> GND
- C4 pad 1: +BATT -> Net-(C3-Pad1)
- C4 pad 2: -BATT -> GND
- C5 pad 2: -BATT -> GND
- C6 pad 2: -BATT -> GND
- C7 pad 2: -BATT -> GND
- C8 pad 1: -BATT -> GND
- C9 pad 1: -BATT -> GND
- DISP1 pad 7: -BATT -> GND
- J1 pad A1: Net-(J1-PadA1) -> GND
- J1 pad A12: Net-(J1-PadA1) -> GND
- J1 pad A4: Net-(J1-PadA4) -> +5V
- J1 pad A5: unconnected-(J1-PadA5) -> Net-(J1-PadA5)
- J1 pad A9: Net-(J1-PadA4) -> +5V
- J1 pad B1: Net-(J1-PadB1) -> GND
- J1 pad B12: Net-(J1-PadB1) -> GND
- J1 pad B4: Net-(J1-PadB4) -> +5V
- J1 pad B5: unconnected-(J1-PadB5) -> Net-(J1-PadB5)
- J1 pad B9: Net-(J1-PadB4) -> +5V
- J2 pad 2: -BATT -> GND
- J4 pad 4: -BATT -> GND
- R2 pad 2: -BATT -> GND
- R3 pad 2: -BATT -> GND
- U1 pad 1: -BATT -> GND
- U1 pad 3: -BATT -> GND
- U1 pad 9: (no net) -> GND
- U2 pad 1: -BATT -> GND
- U2 pad 15: -BATT -> GND
- U2 pad 25: unconnected-(U2-Pad25) -> Net-(C16-Pad1)
- U2 pad 3: +3V3 -> Net-(C15-Pad2)
- U2 pad 38: -BATT -> GND
- U2 pad 39: -BATT -> GND
- U3 pad 2: +BATT -> Net-(C3-Pad1)
- U3 pad 4: -BATT -> GND
- U3 pad 9: (no net) -> GND
- U4 pad 3: -BATT -> GND
Routing:
- net +5V: track 0.00 -> 5.15 mm
- net Net-(J1-PadB5): track 0.00 -> 4.22 mm
- net Net-(J1-PadA5): track 0.00 -> 2.19 mm
- added copper zone on B.Cu, net GND
- added copper zone on F.Cu, net GND
Other:
- outline, holes or cut-outs redrawn

Commit message: placement
Parts:
- removed R21: 0, Resistor_SMD:R_0603_1608Metric
- removed SW7: SW_PWR, Button_Switch_SMD:SW_Push_1P1T_NO_6x6mm_H9.5mm
- R16: value 10k -> 0
- moved DISP1 105.8 mm to (64.5, 49.6)
- moved J1 99.8 mm to (126.2, 74.2), turned to 90 degrees
- moved J3 93.1 mm to (32.9, 53.1), turned to 0 degrees
- moved U4 82.5 mm to (37.2, 55.0), turned to 180 degrees
- moved C9 81.4 mm to (37.8, 51.4), turned to 180 degrees
- moved C10 80.1 mm to (38.5, 49.3), turned to 180 degrees
- moved R8 69.5 mm to (117.3, 57.5), turned to 180 degrees
- moved Q1 69.5 mm to (118.2, 54.8), turned to -90 degrees
- moved R14 67.0 mm to (60.5, 69.1), turned to -90 degrees
- moved R12 66.8 mm to (56.4, 69.1)
- moved R6 65.4 mm to (118.3, 52.0), turned to 180 degrees
- moved SW3 64.1 mm to (52.5, 74.0)
- moved Q2 62.6 mm to (115.0, 54.8), turned to -90 degrees
- moved J2 62.3 mm to (15.1, 108.0)
- moved SW5 61.2 mm to (64.5, 74.0)
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Connections:
- D1 pad 1: Net-(D1-Pad1) -> ENC_S1
- D1 pad 2: PWR_READ -> ENC_BTN
- D2 pad 1: Net-(D1-Pad1) -> ENC_S1
- R16 pad 1: +3V3 -> ENC_BTN
- R16 pad 2: ENC_BTN -> ENC_S1
- R20 pad 2: PWR_READ -> ENC_BTN
- SW4 pad S1: ENC_BTN -> ENC_S1
- U1 pad 9: GND -> (no net)
- U3 pad 9: GND -> (no net)
Routing:
- net unconnected-(DISP1-Pad1): track 0.00 -> 54.5 mm
- net unconnected-(DISP1-Pad2): track 0.00 -> 51.4 mm
- net unconnected-(DISP1-Pad3): track 0.00 -> 47.0 mm
- net unconnected-(DISP1-Pad4): track 0.00 -> 44.0 mm
- net unconnected-(DISP1-Pad5): track 0.00 -> 40.7 mm
- net +3V3: track 0.00 -> 37.2 mm
- net Net-(C15-Pad2): track 0.00 -> 30.0 mm
- net ENC_B: track 0.00 -> 14.4 mm
- net Net-(C16-Pad1): track 0.00 -> 13.9 mm
- net ENC_A: track 0.00 -> 8.89 mm
- net ENC_BTN: track 0.00 -> 7.49 mm
- net ENC_S1: track 0.00 -> 7.09 mm
- net Net-(D2-Pad2): track 0.00 -> 5.28 mm
- net +5V: track 5.15 -> 0.00 mm
- net Net-(J1-PadB5): track 4.22 -> 0.00 mm
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Other:
- outline, holes or cut-outs redrawn

Commit message: placement (possibly close to final)
Parts:
- moved J2 119.3 mm to (126.4, 65.1)
- moved C2 102.3 mm to (117.7, 68.0), turned to -90 degrees
- moved R10 99.5 mm to (120.0, 73.4), turned to 180 degrees
- moved R9 97.5 mm to (120.0, 75.2), turned to 180 degrees
- moved C1 92.7 mm to (115.5, 77.9), turned to 180 degrees
- moved U1 91.7 mm to (113.8, 70.7), turned to 90 degrees
- moved R3 85.1 mm to (111.6, 77.5), turned to 180 degrees
- moved J5 77.1 mm to (100.1, 69.6), turned to -90 degrees
- moved R19 60.1 mm to (107.5, 67.5), turned to -90 degrees
- moved Q4 58.2 mm to (104.8, 66.8), turned to 0 degrees
- moved C3 55.1 mm to (94.2, 76.3), turned to -90 degrees
- moved R17 54.0 mm to (107.5, 71.7), turned to 90 degrees
- moved Q3 53.0 mm to (104.9, 70.0), turned to 0 degrees
- moved C4 52.0 mm to (92.2, 75.3), turned to -90 degrees
- moved L1 52.0 mm to (92.8, 72.5), turned to 90 degrees
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Routing:
- net +BATT: track 1.77 -> 51.8 mm
- net +5V: track 0.00 -> 43.7 mm
- net unconnected-(DISP1-Pad3): track 47.0 -> 13.0 mm
- net unconnected-(DISP1-Pad1): track 54.5 -> 20.6 mm
- net unconnected-(DISP1-Pad2): track 51.4 -> 18.7 mm
- net unconnected-(DISP1-Pad4): track 44.0 -> 12.2 mm
- net unconnected-(DISP1-Pad5): track 40.7 -> 16.4 mm
- net Net-(C3-Pad1): track 0.00 -> 19.3 mm
- net ENC_B: track 14.4 -> 2.10 mm
- net BTN_3: track 0.00 -> 10.1 mm
- net BTN_1: track 0.00 -> 9.81 mm
- net BTN_2: track 0.00 -> 9.79 mm
- net Net-(D2-Pad2): track 5.28 -> 13.2 mm, vias 0 -> 2
- net Net-(Q1-Pad2): track 0.00 -> 5.25 mm
- net Net-(J1-PadB5): track 0.00 -> 3.96 mm
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
Commit message: placement and some routing
Parts:
- moved J2 0.91 mm to (126.3, 66.0)
- moved R17 0.69 mm to (107.0, 72.1)
- moved R18 0.45 mm to (104.7, 72.9)
- moved R4 0.10 mm to (81.6, 72.2)
Routing:
- net +3V3: track 40.6 -> 44.9 mm
- net Net-(J3-Pad1): track 0.00 -> 3.35 mm
- net Net-(J3-Pad2): track 0.00 -> 3.24 mm
- net +5V: track 43.7 -> 43.2 mm
- net PWR_CTRL: track 1.99 -> 1.49 mm

Commit message: routing
Parts:
- added R21: 100k, Resistor_SMD:R_0603_1608Metric, F.Cu at (42.8, 54.2)
- added R22: 100k, Resistor_SMD:R_0603_1608Metric, F.Cu at (40.7, 54.2)
- moved R14 10.1 mm to (59.8, 71.4)
- moved R13 5.09 mm to (95.6, 38.6), turned to -90 degrees
- moved R11 5.04 mm to (90.6, 38.7), turned to -90 degrees
- moved R12 2.77 mm to (47.9, 71.4)
- moved R15 1.22 mm to (71.8, 71.5), turned to -90 degrees
- moved J1 0.20 mm to (126.0, 74.2)
Connections:
- U2 pad 11: unconnected-(U2-Pad11) -> I2S_SD_MODE
- U2 pad 12: unconnected-(U2-Pad12) -> I2S_DIN
- U2 pad 13: unconnected-(U2-Pad13) -> I2S_BCLK
- U2 pad 14: unconnected-(U2-Pad14) -> I2S_LRCLK
- U2 pad 16: unconnected-(U2-Pad16) -> ENC_BTN
- U2 pad 23: unconnected-(U2-Pad23) -> ADC_ENABLE
- U2 pad 24: unconnected-(U2-Pad24) -> ADC IN
- U4 pad 1: unconnected-(U4-Pad1) -> I2S_DIN
- U4 pad 14: unconnected-(U4-Pad14) -> I2S_LRCLK
- U4 pad 16: unconnected-(U4-Pad16) -> I2S_BCLK
- U4 pad 2: unconnected-(U4-Pad2) -> Net-(U4-Pad2)
- U4 pad 4: unconnected-(U4-Pad4) -> I2S_SD_MODE
Routing:
- net I2S_LRCLK: track 0.00 -> 75.8 mm
- net I2S_DIN: track 0.00 -> 72.6 mm
- net I2S_BCLK: track 0.00 -> 72.5 mm
- net I2S_SD_MODE: track 0.00 -> 70.4 mm
- net +3V3: track 44.9 -> 111.0 mm
- net unconnected-(DISP1-Pad3): track 13.0 -> 63.0 mm
- net unconnected-(DISP1-Pad4): track 12.2 -> 61.1 mm
- net unconnected-(DISP1-Pad1): track 20.6 -> 67.7 mm
- net unconnected-(DISP1-Pad2): track 18.7 -> 65.1 mm
- net unconnected-(DISP1-Pad5): track 16.4 -> 58.5 mm
- net ENC_B: track 2.10 -> 23.7 mm
- net ENC_BTN: track 10.6 -> 26.9 mm
- net ADC_ENABLE: track 0.00 -> 9.08 mm
- net Net-(U4-Pad2): track 0.00 -> 4.26 mm
- net ENC_A: track 8.89 -> 13.1 mm
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
Commit message: routing
Parts:
- moved R12 1.70 mm to (48.0, 73.1), turned to 90 degrees
- moved R14 1.70 mm to (59.9, 73.1), turned to 90 degrees
- moved R15 1.70 mm to (71.8, 73.2), turned to 90 degrees
- moved R13 1.30 mm to (95.6, 39.9)
- moved R22 0.63 mm to (41.3, 54.0)
- moved R10 0.36 mm to (119.7, 73.6)
- moved R9 0.30 mm to (119.7, 75.2)
- moved R21 0.28 mm to (43.0, 54.0)
Connections:
- DISP1 pad 1: unconnected-(DISP1-Pad1) -> OLED_RST
- DISP1 pad 2: unconnected-(DISP1-Pad2) -> OLED_DC
- DISP1 pad 3: unconnected-(DISP1-Pad3) -> OLED_CS
- DISP1 pad 4: unconnected-(DISP1-Pad4) -> OLED_CLK
- DISP1 pad 5: unconnected-(DISP1-Pad5) -> OLED_MOSI
- J1 pad S1: Net-(J1-PadS1) -> unconnected-(J1-PadS1)
- J1 pad S2: Net-(J1-PadS1) -> unconnected-(J1-PadS1)
- J1 pad S3: Net-(J1-PadS1) -> unconnected-(J1-PadS1)
- J1 pad S4: Net-(J1-PadS1) -> unconnected-(J1-PadS1)
- U1 pad 6: unconnected-(U1-Pad6) -> STBY
- U1 pad 7: unconnected-(U1-Pad7) -> CHRG
- U2 pad 10: unconnected-(U2-Pad10) -> OLED_RST
- U2 pad 26: unconnected-(U2-Pad26) -> BTN_3
- U2 pad 27: unconnected-(U2-Pad27) -> BTN_2
- U2 pad 28: unconnected-(U2-Pad28) -> BTN_1
- U2 pad 29: unconnected-(U2-Pad29) -> CHRG
- U2 pad 30: unconnected-(U2-Pad30) -> STBY
- U2 pad 4: unconnected-(U2-Pad4) -> ENC_B
- U2 pad 5: unconnected-(U2-Pad5) -> ENC_A
- U2 pad 6: unconnected-(U2-Pad6) -> OLED_MOSI
- U2 pad 7: unconnected-(U2-Pad7) -> OLED_CLK
- U2 pad 8: unconnected-(U2-Pad8) -> OLED_CS
- U2 pad 9: unconnected-(U2-Pad9) -> OLED_DC
Routing:
- net unconnected-(DISP1-Pad1): track 67.7 -> 0.00 mm
- net OLED_RST: track 0.00 -> 67.4 mm
- net OLED_DC: track 0.00 -> 65.2 mm
- net unconnected-(DISP1-Pad2): track 65.1 -> 0.00 mm
- net OLED_CS: track 0.00 -> 63.1 mm
- net unconnected-(DISP1-Pad3): track 63.0 -> 0.00 mm
- net unconnected-(DISP1-Pad4): track 61.1 -> 0.00 mm
- net OLED_CLK: track 0.00 -> 60.7 mm
- net +3V3: track 111.0 -> 170.2 mm, vias 0 -> 2
- net OLED_MOSI: track 0.00 -> 58.5 mm
- net unconnected-(DISP1-Pad5): track 58.5 -> 0.00 mm
- net STBY: track 0.00 -> 38.1 mm, vias 0 -> 2
- net CHRG: track 0.00 -> 36.1 mm, vias 0 -> 2
- net ENC_B: track 23.7 -> 21.4 mm, vias 0 -> 1
- net BTN_3: track 7.95 -> 9.93 mm
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Other:
- board text added: "BOOT"
- board text added: "RST"

Commit message: routing
Parts:
- moved Q3 2.00 mm to (104.9, 72.0)
- moved Q4 2.00 mm to (104.8, 68.8)
- moved R17 2.00 mm to (107.0, 74.1)
- moved R18 2.00 mm to (104.7, 74.9)
- moved R19 2.00 mm to (107.5, 69.5)
- moved J2 1.20 mm to (126.3, 67.2)
- moved SW1 0.54 mm to (123.6, 55.4)
- moved C11 0.50 mm to (89.5, 70.3)
- moved C12 0.50 mm to (89.5, 67.7)
- moved C1 0.41 mm to (115.6, 77.5)
- moved C16 0.40 mm to (124.6, 48.0)
- moved C4 0.33 mm to (92.2, 75.6)
- moved R3 0.30 mm to (111.6, 77.2)
- moved J3 0.21 mm to (33.1, 53.1)
- moved U1 0.20 mm to (113.8, 70.5)
Connections:
- U1 pad 9: (no net) -> GND
- U2 pad 26: BTN_3 -> BTN_2
- U2 pad 27: BTN_2 -> BTN_3
- U2 pad 28: BTN_1 -> PWR_CTRL
- U2 pad 29: CHRG -> BTN_1
- U2 pad 30: STBY -> CHRG
- U2 pad 31: unconnected-(U2-Pad31) -> STBY
- U3 pad 9: (no net) -> GND
Routing:
- net BTN_1: track 10.1 -> 105.4 mm, vias 0 -> 2
- net BTN_2: track 9.92 -> 98.5 mm, vias 0 -> 2
- net BTN_3: track 9.93 -> 88.5 mm, vias 0 -> 2
- net PWR_CTRL: track 1.49 -> 53.6 mm, vias 0 -> 2
- net +3V3: track 170.2 -> 212.7 mm
- net GND: track 0.00 -> 41.2 mm, vias 1 -> 49
- net CHRG: track 36.1 -> 42.7 mm
- net STBY: track 38.1 -> 44.1 mm
- net +BATT: track 52.0 -> 54.4 mm
- net Net-(C16-Pad1): track 13.9 -> 15.6 mm
- net Net-(C3-Pad1): track 19.3 -> 18.0 mm
- net ADC_ENABLE: track 9.08 -> 10.1 mm
- net Net-(D2-Pad2): track 13.2 -> 13.8 mm
- net +5V: track 42.9 -> 42.4 mm
- added copper zone on B.Cu, net (none)
- added copper zone on F.Cu, net (none)
- removed copper zone on B.Cu, net GND
- removed copper zone on F.Cu, net GND
